File: eagle/oresat0-plusz-end-cap.sch (EAGLE design)
At the start: 31 parts, among them U1 LTC4305, U2 MMC5883MA, U3 MMC5883MA

Commit message: Removed connector cutout from board outline. Increased restrict area for turnstile antenna. Changed some traces to the top layer to avoid the bstop area, and the new restrict area. Added NP resistors connecting magnetometer interrupts to i2c buffer alert inputs. Moved components away from backplane.
Parts:
- added R11, R12: 4.7k, oresat-rcl:R-US_0603-B-NOSILK
Connections:
- new net N$10: R12.1, U2.INT
- new net N$7: R11.1, U3.INT
- net N$4: now also R11.2
- net N$6: now also R12.2
Changed lines of the file:
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@@
 <part name="TP4" library="oresat-misc" deviceset="TEST-POINT-LARGE-SQUARE" device=""/>
 <part name="TP5" library="oresat-misc" deviceset="TEST-POINT-LARGE-SQUARE" device=""/>
+<part name="R11" library="oresat-rcl" deviceset="R-US_" device="0603-B-NOSILK" value="4.7k">
+<attribute name="DIS" value="Digi-Key"/>
+<attribute name="DPN" value="1276-4275-1-ND"/>
+<attribute name="MFR" value="Samsung"/>
+<attribute name="MPN" value="RC1005F6653CS"/>
+</part>
+<part name="R12" library="oresat-rcl" deviceset="R-US_" device="0603-B-NOSILK" value="4.7k">
+<attribute name="DIS" value="Digi-Key"/>
+<attribute name="DPN" value="1276-4275-1-ND"/>
+<attribute name="MFR" value="Samsung"/>
+<attribute name="MPN" value="RC1005F6653CS"/>
+</part>
 </parts>
 <sheets>
@@
 <attribute name="NAME" x="116.84" y="162.56" size="1.778" layer="104"/>
 </instance>
-<instance part="TP7" gate="G$1" x="111.76" y="138.43" smashed="yes">
-<attribute name="NAME" x="109.22" y="140.97" size="1.778" layer="104"/>
+<instance part="TP7" gate="G$1" x="111.76" y="152.4" smashed="yes">
+<attribute name="NAME" x="113.03" y="151.13" size="1.778" layer="104"/>
 </instance>
 <instance part="TP8" gate="G$1" x="104.14" y="128.27" smashed="yes">
@@
 <instance part="TP5" gate="G$1" x="233.68" y="95.25" smashed="yes">
 <attribute name="NAME" x="232.41" y="91.44" size="1.27" layer="104"/>
+</instance>
+<instance part="R11" gate="R" x="246.38" y="152.4" smashed="yes" rot="R180">
+<attribute name="DIS" x="246.38" y="152.4" size="1.778" layer="96" rot="R180" display="off"/>
+<attribute name="DPN" x="246.38" y="152.4" size="1.778" layer="96" rot="R180" display="off"/>
+<attribute name="MFR" x="246.38" y="152.4" size="1.778" layer="96" rot="R180" display="off"/>
+<attribute name="MPN" x="246.38" y="152.4" size="1.778" layer="96" rot="R180" display="off"/>
+<attribute name="NAME" x="250.19" y="150.9014" size="1.778" layer="95" rot="R180"/>
+<attribute name="VALUE" x="245.11" y="151.13" size="1.778" layer="96" rot="R180"/>
+</instance>
+<instance part="R12" gate="R" x="246.38" y="90.17" smashed="yes" rot="R180">
+<attribute name="DIS" x="246.38" y="90.17" size="1.778" layer="96" rot="R180" display="off"/>
+<attribute name="DPN" x="246.38" y="90.17" size="1.778" layer="96" rot="R180" display="off"/>
+<attribute name="MFR" x="246.38" y="90.17" size="1.778" layer="96" rot="R180" display="off"/>
+<attribute name="MPN" x="246.38" y="90.17" size="1.778" layer="96" rot="R180" display="off"/>
+<attribute name="NAME" x="250.19" y="88.6714" size="1.778" layer="95" rot="R180"/>
+<attribute name="VALUE" x="245.11" y="88.9" size="1.778" layer="96" rot="R180"/>
 </instance>
 </instances>
@@
 <segment>
 <pinref part="SUPPLY6" gate="G$1" pin="3.3V"/>
-<wire x1="111.76" y1="165.1" x2="111.76" y2="138.43" width="0.1524" layer="91"/>
+<wire x1="111.76" y1="165.1" x2="111.76" y2="152.4" width="0.1524" layer="91"/>
 <wire x1="96.52" y1="149.86" x2="111.76" y2="149.86" width="0.1524" layer="91"/>
 <pinref part="C4" gate="CE" pin="1"/>
 <wire x1="111.76" y1="132.08" x2="111.76" y2="149.86" width="0.1524" layer="91"/>
 <label x="96.52" y="149.86" size="1.778" layer="95"/>
-<wire x1="111.76" y1="138.43" x2="111.76" y2="149.86" width="0.1524" layer="91"/>
-<junction x="111.76" y="138.43"/>
+<wire x1="111.76" y1="152.4" x2="111.76" y2="149.86" width="0.1524" layer="91"/>
+<junction x="111.76" y="152.4"/>
 <junction x="111.76" y="149.86"/>
 <pinref part="CF2" gate="G$1" pin="6"/>
@@
 <pinref part="TP4" gate="G$1" pin="1"/>
 <junction x="229.87" y="97.79"/>
+<junction x="218.44" y="97.79"/>
 </segment>
 </net>
@@
 <wire x1="198.12" y1="154.94" x2="198.12" y2="162.56" width="0.1524" layer="91"/>
 <pinref part="R3" gate="R" pin="1"/>
+<pinref part="R11" gate="R" pin="2"/>
+<wire x1="241.3" y1="152.4" x2="214.63" y2="152.4" width="0.1524" layer="91"/>
+<wire x1="214.63" y1="152.4" x2="214.63" y2="154.94" width="0.1524" layer="91"/>
+<wire x1="214.63" y1="154.94" x2="198.12" y2="154.94" width="0.1524" layer="91"/>
+<junction x="198.12" y="154.94"/>
 </segment>
 </net>
@@
 <wire x1="203.2" y1="144.78" x2="203.2" y2="162.56" width="0.1524" layer="91"/>
 <pinref part="R8" gate="R" pin="1"/>
+<pinref part="R12" gate="R" pin="2"/>
+<wire x1="241.3" y1="90.17" x2="207.01" y2="90.17" width="0.1524" layer="91"/>
+<wire x1="207.01" y1="90.17" x2="207.01" y2="144.78" width="0.1524" layer="91"/>
+<wire x1="207.01" y1="144.78" x2="203.2" y2="144.78" width="0.1524" layer="91"/>
+<junction x="203.2" y="144.78"/>
 </segment>
 </net>
@@
 </segment>
 </net>
+<net name="N$7" class="0">
+<segment>
+<pinref part="U3" gate="G$1" pin="INT"/>
+<pinref part="R11" gate="R" pin="1"/>
+<wire x1="276.86" y1="152.4" x2="251.46" y2="152.4" width="0.1524" layer="91"/>
+</segment>
+</net>
+<net name="N$10" class="0">
+<segment>
+<pinref part="U2" gate="G$1" pin="INT"/>
+<pinref part="R12" gate="R" pin="1"/>
+<wire x1="276.86" y1="90.17" x2="251.46" y2="90.17" width="0.1524" layer="91"/>
+</segment>
+</net>

Commit message: v1.0 end caps for OreSat0!
Parts:
- R11, R12: value 4.7k -> NP
- U1: value LTC4305 -> LTC4305IGN
Other:
- note added: "1.0"
- note removed: "2.0"
Changed lines of the file:
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@@
 <?xml version="1.0" encoding="utf-8"?>
 <!DOCTYPE eagle SYSTEM "eagle.dtd">
-<eagle version="9.5.1">
+<eagle version="9.6.1">
 <drawing>
 <settings>
@@
 <setting verticaltext="up"/>
 </settings>
-<grid distance="0.05" unitdist="inch" unit="inch" style="lines" multiple="1" display="no" altdistance="0.01" altunitdist="inch" altunit="inch"/>
+<grid distance="0.1" unitdist="inch" unit="inch" style="lines" multiple="1" display="no" altdistance="0.01" altunitdist="inch" altunit="inch"/>
 <layers>
 <layer number="1" name="Top" color="4" fill="1" visible="no" active="no"/>
@@
 </part>
 <part name="GND9" library="supply1" deviceset="GND" device=""/>
-<part name="U1" library="U-Linear-LTC4305-2-Channel-Bus-Multiplexer" deviceset="LTC4305" device=""/>
+<part name="U1" library="U-Linear-LTC4305-2-Channel-Bus-Multiplexer" deviceset="LTC4305" device="" value="LTC4305IGN"/>
 <part name="GND12" library="supply1" deviceset="GND" device=""/>
 <part name="GND13" library="supply1" deviceset="GND" device=""/>
@@
 <part name="TP4" library="oresat-misc" deviceset="TEST-POINT-LARGE-SQUARE" device=""/>
 <part name="TP5" library="oresat-misc" deviceset="TEST-POINT-LARGE-SQUARE" device=""/>
-<part name="R11" library="oresat-rcl" deviceset="R-US_" device="0603-B-NOSILK" value="4.7k">
-<attribute name="DIS" value="Digi-Key"/>
-<attribute name="DPN" value="1276-4275-1-ND"/>
-<attribute name="MFR" value="Samsung"/>
-<attribute name="MPN" value="RC1005F6653CS"/>
-</part>
-<part name="R12" library="oresat-rcl" deviceset="R-US_" device="0603-B-NOSILK" value="4.7k">
+<part name="R11" library="oresat-rcl" deviceset="R-US_" device="0603-B-NOSILK" value="NP">
+<attribute name="DIS" value="Digi-Key"/>
+<attribute name="DPN" value="1276-4275-1-ND"/>
+<attribute name="MFR" value="Samsung"/>
+<attribute name="MPN" value="RC1005F6653CS"/>
+</part>
+<part name="R12" library="oresat-rcl" deviceset="R-US_" device="0603-B-NOSILK" value="NP">
 <attribute name="DIS" value="Digi-Key"/>
 <attribute name="DPN" value="1276-4275-1-ND"/>
@@
 <plain>
 <text x="341.63" y="26.67" size="3.81" layer="94">OreSat0 +Z End Cap</text>
-<text x="416.56" y="6.35" size="3.81" layer="94">2.0</text>
+<text x="416.56" y="6.35" size="3.81" layer="94">1.0</text>
 <text x="11.43" y="5.08" size="1.778" layer="97">All resistors 0402 +/- 1% unless marked</text>
 <text x="11.43" y="2.54" size="1.778" layer="97">All caps are 0402 ceramic 10% X5R Vw&gt;=16V unless marked</text>

Commit message: Added BOMs and updated attributes for OreSat0 + and - Z end caps.
Parts:
- C1, C10, C2, C3, C7: DPN 1276-1001-1-ND -> 1276-CL10B104KB8NNNLCT-ND; MPN CL05B104KO5NNNC -> CL10B104KB8NNNL
- C12, C13, C4: DPN 1276-1001-1-ND -> 490-14461-1-ND; MFR Samsung -> Murata; MPN CL05B104KO5NNNC -> GRM188D71A106KA73D
- CF2: DIS (none) -> Digi-Key; DPN (none) -> A122888-ND; MFR (none) -> Harwin; MPN (none) -> M55-7011242R
- D2: DIS (none) -> Digi-Key; DPN (none) -> 511-1584-1-ND; MFR (none) -> Rohn; MPN (none) -> SML-E12M8WT86
- R1, R10, R3, R4, R5, R6, R7, R8, R9: DPN 1276-4275-1-ND -> A129696CT-ND; MFR Samsung -> TE Connectivity; MPN RC1005F6653CS -> CRGCQ0603F4K7
- R11, R12: DIS Digi-Key -> (none); DPN 1276-4275-1-ND -> (none); MFR Samsung -> (none); MPN RC1005F6653CS -> (none)
- R2: DPN 1276-4275-1-ND -> A129693CT-ND; MFR Samsung -> TE Connectivity; MPN RC1005F6653CS -> CRGCQ0603F2K7
- U1: DIS (none) -> Digi-Key; DPN (none) -> LTC4305IGN#PBF-ND; MFR (none) -> Analog; MPN (none) -> LTC4305IGN#PBF
- U2, U3: DIS (none) -> Digi-Key; DPN (none) -> 1267-1072-1-ND; MFR (none) -> Memsic; MPN (none) -> MMC5883MA
