File: eagle/oresat0-plusz-end-cap.sch (EAGLE design)
At the start: 33 parts, among them U1 LTC4305IGN, U2 MMC5883MA, U3 MMC5883MA

Commit message: New +Z end cap with larger cutout for turnstile.
New -Z end cap with amazing artwork from Jennifer and thank yous.
Other:
- note added: "1.1"
- note removed: "1.0"
Changed lines of the file:
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@@
 <drawing>
 <settings>
-<setting alwaysvectorfont="yes"/>
+<setting alwaysvectorfont="no"/>
 <setting keepoldvectorfont="yes"/>
 <setting verticaltext="up"/>
@@
 <plain>
 <text x="341.63" y="26.67" size="3.81" layer="94">OreSat0 +Z End Cap</text>
-<text x="416.56" y="6.35" size="3.81" layer="94">1.0</text>
+<text x="416.56" y="6.35" size="3.81" layer="94">1.1</text>
 <text x="11.43" y="5.08" size="1.778" layer="97">All resistors 0402 +/- 1% unless marked</text>
 <text x="11.43" y="2.54" size="1.778" layer="97">All caps are 0402 ceramic 10% X5R Vw&gt;=16V unless marked</text>
