File: eagle/oresat0-plusz-end-cap.brd (EAGLE design)
At the start: 105.6 x 105.6 mm, 33 parts, among them U1 LTC4305IGN, U2 MMC5883MA, U3 MMC5883MA

Commit message: New +Z end cap with larger cutout for turnstile.
New -Z end cap with amazing artwork from Jennifer and thank yous.
Other:
- board text added: "2021/04/06"
- board text added: "OreSat0 +Z End Cap v1.1"
- board text removed: "2020/08/28"
- board text removed: "OreSat0 +Z End Cap v1.0"
