File: oresat0.5-plusz-end-cap/oresat0.5-plusz-end-cap.kicad_sch (KiCad schematic)
At the start: 33 parts

Commit message: Updated oresat0.5 +Z board outline
Parts:
- C1, C10, C12, C13, C2, C3, C4, C7, R1, R10, R2, R3, R4, R5, R6, R7, R8, R9: footprint (none) -> oresat0.5-plusz-end-cap:.0603-B-NOSILK
- CF2: footprint (none) -> oresat0-plusz-end-cap:HARWIN-M55-70X1242R
- D2: footprint (none) -> oresat0-plusz-end-cap:LED-0603
- R11, R12: value (none) -> NP; footprint (none) -> oresat0.5-plusz-end-cap:.0603-B-NOSILK
- TP1, TP2, TP3, TP4, TP5, TP6, TP7, TP8: value (none) -> TEST-POINT-LARGE-SQUARE; footprint (none) -> oresat0-plusz-end-cap:1X01
- U1: footprint (none) -> oresat0-plusz-end-cap:16-SSOP
- U2, U3: footprint (none) -> oresat0-plusz-end-cap:LGA-16(3X3)
Other:
- note removed: "All caps are 0402 ceramic 10% X5R Vw>=16V unless marked"
- note removed: "All resistors 0402 +/- 1% unless marked"

Commit message: Updated both oresat0.5 end caps. Fixed layout, and added patch antennas
Parts:
- added ANT1: ANT1008, oresat-misc:RFMi-ANT1008-S-Band-Patch, symbol Device:Antenna_Shield
- added J2: U.FL-R-SMA, Connector_Coaxial:U.FL_Hirose_U.FL-R-SMT-1_Vertical, symbol Connector:Conn_Coaxial
- renumbered CF2 to J1
Connections:
- net GND: now also ANT1.2 (Shield), J2.2 (Ext)
- new net: ANT1.1 (A), J2.1 (In)
Other:
- note added: "1.0"
- note added: "OreSat0.5 +Z End Cap"
- note removed: "1.1"
- note removed: "OreSat0 +Z End Cap"
Changed lines of the file:
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@@
+    (stroke (width 0) (type default) (color 0 0 0 0))
+  )
+  (wire (pts (xy 144.78 91.44) (xy 144.78 93.98))
     (stroke (width 0) (type default) (color 0 0 0 0))
   )
@@
     (stroke (width 0) (type default) (color 0 0 0 0))
   )
+  (wire (pts (xy 147.32 91.44) (xy 147.32 93.98))
+    (stroke (width 0) (type default) (color 0 0 0 0))
+  )
   (wire (pts (xy 114.3 152.4) (xy 114.3 154.94))
     (stroke (width 0) (type default) (color 0 0 0 0))
   )
+  (wire (pts (xy 137.16 93.98) (xy 144.78 93.98))
+    (stroke (width 0) (type default) (color 0 0 0 0))
+  )
   (wire (pts (xy 218.44 121.92) (xy 220.98 121.92))
     (stroke (width 0) (type default) (color 0 0 0 0))
@@
   )
   (wire (pts (xy 236.22 134.62) (xy 236.22 139.7))
+    (stroke (width 0) (type default) (color 0 0 0 0))
+  )
+  (wire (pts (xy 132.08 99.06) (xy 132.08 101.6))
     (stroke (width 0) (type default) (color 0 0 0 0))
   )
@@
     (effects (font (size 1.778 1.5113)) (justify left bottom))
   )
-  (text "1.1" (at 434.34 290.83 180)
+  (text "1.0" (at 434.34 290.83 180)
     (effects (font (size 3.81 3.2385)) (justify left bottom))
   )
-  (text "OreSat0 +Z End Cap" (at 359.41 270.51 180)
+  (text "OreSat0.5 +Z End Cap" (at 359.41 270.51 180)
     (effects (font (size 3.81 3.2385)) (justify left bottom))
   )
@@
     (pin "1")
   )
+  (symbol (lib_id "oresat0-plusz-end-cap-eagle-import:GND") (at 132.08 104.14 0) (mirror y) (unit 1)
+    (in_bom yes) (on_board yes)
+    (property "Reference" "#GND0102" (id 0) (at 132.08 104.14 0)
+      (effects (font (size 1.27 1.27)) hide)
+    )
+    (property "Value" "GND" (id 1) (at 134.62 106.68 0)
+      (effects (font (size 1.778 1.5113)) (justify left bottom))
+    )
+    (property "Footprint" "oresat0-plusz-end-cap:" (id 2) (at 132.08 104.14 0)
+      (effects (font (size 1.27 1.27)) hide)
+    )
+    (property "Datasheet" "" (id 3) (at 132.08 104.14 0)
+      (effects (font (size 1.27 1.27)) hide)
+    )
+    (pin "1")
+  )
   (symbol (lib_id "oresat0-plusz-end-cap-eagle-import:GND") (at 121.92 177.8 0) (mirror y) (unit 1)
     (in_bom yes) (on_board yes)
@@
     (property "Value" "" (id 4) (at 241.3 191.77 0)
       (effects (font (size 1.778 1.5113)) (justify left bottom) hide)
+    )
+    (pin "1")
+    (pin "2")
+  )
+  (symbol (lib_id "Device:Antenna_Shield") (at 144.78 86.36 0) (unit 1)
+    (in_bom yes) (on_board yes) (fields_autoplaced)
+    (property "Reference" "ANT1" (id 0) (at 148.59 84.4549 0)
+      (effects (font (size 1.27 1.27)) (justify left))
+    )
+    (property "Value" "ANT1008" (id 1) (at 148.59 86.9949 0)
+      (effects (font (size 1.27 1.27)) (justify left))
+    )
+    (property "Footprint" "oresat-misc:RFMi-ANT1008-S-Band-Patch" (id 2) (at 144.78 83.82 0)
+      (effects (font (size 1.27 1.27)) hide)
+    )
+    (property "Datasheet" "~" (id 3) (at 144.78 83.82 0)
+      (effects (font (size 1.27 1.27)) hide)
     )
     (pin "1")
@@
     (pin "1")
   )
+  (symbol (lib_id "oresat0-plusz-end-cap-eagle-import:GND") (at 147.32 96.52 0) (mirror y) (unit 1)
+    (in_bom yes) (on_board yes)
+    (property "Reference" "#GND0101" (id 0) (at 147.32 96.52 0)
+      (effects (font (size 1.27 1.27)) hide)
+    )
+    (property "Value" "GND" (id 1) (at 149.86 99.06 0)
+      (effects (font (size 1.778 1.5113)) (justify left bottom))
+    )
+    (property "Footprint" "oresat0-plusz-end-cap:" (id 2) (at 147.32 96.52 0)
+      (effects (font (size 1.27 1.27)) hide)
+    )
+    (property "Datasheet" "" (id 3) (at 147.32 96.52 0)
+      (effects (font (size 1.27 1.27)) hide)
+    )
+    (pin "1")
+  )
   (symbol (lib_id "oresat0-plusz-end-cap-eagle-import:TEST-POINT-LARGE-SQUARE") (at 137.16 137.16 0) (unit 1)
     (in_bom yes) (on_board yes)
@@
     )
     (property "Datasheet" "" (id 3) (at 264.16 207.01 0)
+      (effects (font (size 1.27 1.27)) hide)
+    )
+    (pin "1")
+    (pin "2")
+  )
+  (symbol (lib_id "Connector:Conn_Coaxial") (at 132.08 93.98 0) (mirror y) (unit 1)
+    (in_bom yes) (on_board yes) (fields_autoplaced)
+    (property "Reference" "J2" (id 0) (at 132.3974 86.36 0))
+    (property "Value" "U.FL-R-SMA" (id 1) (at 132.3974 88.9 0))
+    (property "Footprint" "Connector_Coaxial:U.FL_Hirose_U.FL-R-SMT-1_Vertical" (id 2) (at 132.08 93.98 0)
+      (effects (font (size 1.27 1.27)) hide)
+    )
+    (property "Datasheet" " ~" (id 3) (at 132.08 93.98 0)
       (effects (font (size 1.27 1.27)) hide)
     )
@@
   (symbol (lib_id "oresat0-plusz-end-cap-eagle-import:J-HARWIN-M55-70X1242R") (at 104.14 149.86 0) (mirror y) (unit 1)
     (in_bom yes) (on_board yes)
-    (property "Reference" "CF2" (id 0) (at 110.49 130.81 0)
+    (property "Reference" "J1" (id 0) (at 110.49 130.81 0)
       (effects (font (size 1.778 1.5113)) (justify left bottom))
     )
@@
       (reference "#GND025") (unit 1) (value "GND") (footprint "oresat0-plusz-end-cap:")
     )
+    (path "/8464bde2-a646-4bf9-8c2f-2ce8f91f03dc"
+      (reference "#GND0101") (unit 1) (value "GND") (footprint "oresat0-plusz-end-cap:")
+    )
+    (path "/03d93d97-befe-4ed5-8af6-319d37e6a38b"
+      (reference "#GND0102") (unit 1) (value "GND") (footprint "oresat0-plusz-end-cap:")
+    )
     (path "/f6b9336a-12e6-4c9c-b65e-e608544f56ed"
       (reference "#SUPPLY01") (unit 1) (value "3.3V") (footprint "oresat0-plusz-end-cap:")
@@
       (reference "#SUPPLY08") (unit 1) (value "3.3V") (footprint "oresat0-plusz-end-cap:")
     )
+    (path "/3ba63093-1664-41b7-8bad-99c8aaf610ef"
+      (reference "ANT1") (unit 1) (value "ANT1008") (footprint "oresat-misc:RFMi-ANT1008-S-Band-Patch")
+    )
     (path "/4a7e51fb-caa1-4542-9483-5dd5d44c807f"
       (reference "C1") (unit 1) (value "100n") (footprint "oresat0.5-plusz-end-cap:.0603-B-NOSILK")
@@
       (reference "C13") (unit 1) (value "10u") (footprint "oresat0.5-plusz-end-cap:.0603-B-NOSILK")
     )
-    (path "/dff41a40-21e0-41b9-aeb3-a577a9604432"
-      (reference "CF2") (unit 1) (value "J-HARWIN-M55-70X1242R") (footprint "oresat0-plusz-end-cap:HARWIN-M55-70X1242R")
-    )
     (path "/2e2f32f8-a7af-4280-a8e8-a2f2ba471a3b"
       (reference "D2") (unit 1) (value "GREEN") (footprint "oresat0-plusz-end-cap:LED-0603")
     )
+    (path "/dff41a40-21e0-41b9-aeb3-a577a9604432"
+      (reference "J1") (unit 1) (value "J-HARWIN-M55-70X1242R") (footprint "oresat0-plusz-end-cap:HARWIN-M55-70X1242R")
+    )
+    (path "/cd812eda-93b6-404b-a98b-394835ee7377"
+      (reference "J2") (unit 1) (value "U.FL-R-SMA") (footprint "Connector_Coaxial:U.FL_Hirose_U.FL-R-SMT-1_Vertical")
+    )
     (path "/5ebf093a-6350-4fb8-a30f-ce3ca8febaaf"

Commit message: Updated both OreSat0.5 end caps and cleaned up errors
Parts:
- C1, C10, C12, C13, C2, C3, C4, C7: symbol oresat0-plusz-end-cap-eagle-import:C-EU0603-B-NOSILK -> oresat0.5-plusz-end-cap-eagle-import:C-EU0603-B-NOSILK
- D2: symbol oresat0-plusz-end-cap-eagle-import:LED-GREEN0603 -> oresat0.5-plusz-end-cap-eagle-import:LED-GREEN0603
- J1: symbol oresat0-plusz-end-cap-eagle-import:J-HARWIN-M55-70X1242R -> oresat0.5-plusz-end-cap-eagle-import:J-HARWIN-M55-70X1242R
- R1, R10, R11, R12, R2, R3, R4, R5, R6, R7, R8, R9: symbol oresat0-plusz-end-cap-eagle-import:R-US_0603-B-NOSILK -> oresat0.5-plusz-end-cap-eagle-import:R-US_0603-B-NOSILK
- TP1, TP2, TP3, TP4, TP5, TP6, TP7, TP8: symbol oresat0-plusz-end-cap-eagle-import:TEST-POINT-LARGE-SQUARE -> oresat0.5-plusz-end-cap-eagle-import:TEST-POINT-LARGE-SQUARE
- U1: value (none) -> LTC4305; symbol oresat0-plusz-end-cap-eagle-import:LTC4305 -> oresat0.5-plusz-end-cap-eagle-import:LTC4305
- U2, U3: symbol oresat0-plusz-end-cap-eagle-import:MMC5883MA -> oresat0.5-plusz-end-cap-eagle-import:MMC5883MA
Connections:
- no-connect marks 0 -> 4
Other:
- moved on the sheet: ANT1, C1, C10, C12, C13, C2, C3, C4, C7, D2, J1, J2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

Commit message: OreSat0.5 end caps design review fixes
Connections:
- net I2C-SCL renamed MAG-SCL
- net I2C-SDA renamed MAG-SDA
Other:
- note added: "0x88"
- note added: "MAG-PWR"
Changed lines of the file:
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@@
   (junction (at 240.03 186.69) (diameter 0) (color 0 0 0 0)
   )
+  (junction (at 114.3 144.78) (diameter 0) (color 0 0 0 0)
+  )
   (junction (at 302.26 162.56) (diameter 0) (color 0 0 0 0)
   )
   (junction (at 233.68 189.23) (diameter 0) (color 0 0 0 0)
-  )
-  (junction (at 99.06 160.02) (diameter 0) (color 0 0 0 0)
   )
   (junction (at 307.34 101.6) (diameter 0) (color 0 0 0 0)
@@
     (stroke (width 0) (type default) (color 0 0 0 0))
   )
+  (wire (pts (xy 114.3 144.78) (xy 114.3 156.21))
+    (stroke (width 0) (type default) (color 0 0 0 0))
+  )
   (wire (pts (xy 228.6 109.22) (xy 228.6 111.76))
     (stroke (width 0) (type default) (color 0 0 0 0))
@@
     (stroke (width 0) (type default) (color 0 0 0 0))
   )
-  (wire (pts (xy 88.9 160.02) (xy 88.9 154.94))
-    (stroke (width 0) (type default) (color 0 0 0 0))
-  )
   (wire (pts (xy 322.58 127) (xy 317.5 127))
     (stroke (width 0) (type default) (color 0 0 0 0))
@@
     (stroke (width 0) (type default) (color 0 0 0 0))
   )
-  (wire (pts (xy 99.06 160.02) (xy 88.9 160.02))
-    (stroke (width 0) (type default) (color 0 0 0 0))
-  )
   (wire (pts (xy 302.26 147.32) (xy 302.26 144.78))
     (stroke (width 0) (type default) (color 0 0 0 0))
@@
     (stroke (width 0) (type default) (color 0 0 0 0))
   )
-  (wire (pts (xy 114.3 139.7) (xy 114.3 156.21))
+  (wire (pts (xy 114.3 139.7) (xy 114.3 144.78))
     (stroke (width 0) (type default) (color 0 0 0 0))
   )
@@
     (stroke (width 0) (type default) (color 0 0 0 0))
   )
+  (wire (pts (xy 116.84 144.78) (xy 114.3 144.78))
+    (stroke (width 0) (type default) (color 0 0 0 0))
+  )
   (wire (pts (xy 172.72 142.24) (xy 172.72 139.7))
     (stroke (width 0) (type default) (color 0 0 0 0))
@@
     (stroke (width 0) (type default) (color 0 0 0 0))
   )
+  (wire (pts (xy 116.84 142.24) (xy 116.84 144.78))
+    (stroke (width 0) (type default) (color 0 0 0 0))
+  )
   (wire (pts (xy 106.68 132.08) (xy 99.06 132.08))
     (stroke (width 0) (type default) (color 0 0 0 0))
@@
   (wire (pts (xy 246.38 127) (xy 228.6 127))
     (stroke (width 0) (type default) (color 0 0 0 0))
+  )
+  (text "0x88" (at 167.64 142.24 0)
+    (effects (font (size 1.27 1.27)) (justify left bottom))
   )
   (text "-X+Y Corner" (at 281.94 210.82 180)
     (effects (font (size 1.778 1.5113)) (justify left bottom))
   )
+  (text "MAG-PWR" (at 106.68 134.62 0)
+    (effects (font (size 1.27 1.27)) (justify left bottom))
+  )
   (text "1.0" (at 19.045 260.231 180)
     (effects (font (size 2.032 2.032)) (justify left bottom))
@@
     (effects (font (size 1.778 1.5113)) (justify left bottom))
   )
-  (label "SDA1" (at 287.02 127 0)
+  (label "SDA1" (at 279.4 127 0)
     (effects (font (size 1.2446 1.2446)) (justify left bottom))
   )
-  (label "I2C-SCL" (at 106.68 129.54 0)
+  (label "MAG-SCL" (at 106.68 129.54 0)
     (effects (font (size 1.2446 1.2446)) (justify left bottom))
   )
@@
     (effects (font (size 1.2446 1.2446)) (justify left bottom))
   )
-  (label "SCL1" (at 287.02 124.46 0)
+  (label "SCL1" (at 279.4 124.46 0)
     (effects (font (size 1.2446 1.2446)) (justify left bottom))
   )
@@
     (effects (font (size 1.2446 1.2446)) (justify left bottom))
   )
-  (label "I2C-SDA" (at 106.68 124.46 0)
+  (label "MAG-SDA" (at 106.68 124.46 0)
     (effects (font (size 1.2446 1.2446)) (justify left bottom))
   )
-  (label "I2C-SDA" (at 160.02 132.08 0)
+  (label "MAG-SDA" (at 160.02 132.08 0)
     (effects (font (size 1.2446 1.2446)) (justify left bottom))
   )
-  (label "3.3V" (at 106.68 134.62 0)
+  (label "3.3V" (at 116.84 134.62 0)
     (effects (font (size 1.2446 1.2446)) (justify left bottom))
   )
@@
     (effects (font (size 1.2446 1.2446)) (justify left bottom))
   )
-  (label "I2C-SCL" (at 160.02 129.54 0)
+  (label "MAG-SCL" (at 160.02 129.54 0)
     (effects (font (size 1.2446 1.2446)) (justify left bottom))
   )
@@
     (pin "2")
   )
-  (symbol (lib_id "power:PWR_FLAG") (at 88.9 154.94 0) (unit 1)
+  (symbol (lib_id "power:PWR_FLAG") (at 116.84 142.24 0) (unit 1)
     (in_bom yes) (on_board yes) (fields_autoplaced)
-    (property "Reference" "#FLG0101" (id 0) (at 88.9 153.035 0)
-      (effects (font (size 1.27 1.27)) hide)
-    )
-    (property "Value" "PWR_FLAG" (id 1) (at 88.9 149.86 0))
-    (property "Footprint" "" (id 2) (at 88.9 154.94 0)
-      (effects (font (size 1.27 1.27)) hide)
-    )
-    (property "Datasheet" "~" (id 3) (at 88.9 154.94 0)
-      (effects (font (size 1.27 1.27)) hide)
-    )
+    (property "Reference" "#FLG0101" (id 0) (at 116.84 140.335 0)
+      (effects (font (size 1.27 1.27)) hide)
+    )
+    (property "Value" "PWR_FLAG" (id 1) (at 116.84 137.16 0))
+    (property "Footprint" "" (id 2) (at 116.84 142.24 0)
+      (effects (font (size 1.27 1.27)) hide)
+    )
+    (property "Datasheet" "~" (id 3) (at 116.84 142.24 0)
+      (effects (font (size 1.27 1.27)) hide)
+    )

Commit message: Updated end caps
Parts:
- J1: footprint oresat0-plusz-end-cap:HARWIN-M55-70X1242R -> oresat0.5-plusz-end-cap:HARWIN-M55-70X1242R
- TP1, TP2, TP3, TP4, TP5, TP6, TP7, TP8: footprint oresat0-plusz-end-cap:1X01 -> oresat-misc:TestPoint-0.75mm-th

Commit message: Updated mounting holes
Parts:
- U2, U3: value (none) -> MMC5883MA
Changed lines of the file:
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@@
       (effects (font (size 1.27 1.27)) hide)
     )
-    (property "Value" "" (at 302.26 127 0)
+    (property "Value" "MMC5883MA" (at 302.26 127 0)
       (effects (font (size 1.778 1.5113)) (justify left bottom) hide)
     )
@@
     (pin "2")
     (pin "9")
+    (pin "12")
+    (pin "14")
+    (pin "3")
+    (pin "4")
+    (pin "5")
+    (pin "6")
+    (pin "7")
+    (pin "8")
     (instances
       (project "oresat0.5-plusz-end-cap"
@@
       (effects (font (size 1.27 1.27)) hide)
     )
-    (property "Value" "" (at 302.26 189.23 0)
+    (property "Value" "MMC5883MA" (at 302.26 189.23 0)
       (effects (font (size 1.778 1.5113)) (justify left bottom) hide)
     )
@@
     (pin "2")
     (pin "9")
-    (instances
-      (project "oresat0.5-plusz-end-cap"
+    (pin "12")
+    (pin "14")
+    (pin "3")
+    (pin "4")
+    (pin "5")
+    (pin "6")
+    (pin "7")
+    (pin "8")
+    (instances
+      (project "oresat0.5-plusz-end-cap"
