File: oresat0.5-plusz-end-cap/oresat0.5-plusz-end-cap.kicad_sch (KiCad schematic)
At the start: 35 parts, among them J1 M55-7011242R, J2 U.FL-R-SMA, U1 LTC4305, U2 MMC5983MA, U3 MMC5983MA

Commit message: Fixed BOM.
Parts:
- ANT1: DPN (none) -> N/A; DST (none) -> N/A; MFR (none) -> RFMi; MPN (none) -> ANT1008
- C1, C10, C2, C3, C7: DPN (none) -> 587-3472-1-ND; DST (none) -> Digi-Key; MFR (none) -> Taiyo Yuden; MPN (none) -> TMK107BJ104KAHT
- C12, C13, C4: DPN (none) -> 490-12317-1-ND; DST (none) -> Digi-Key; MFR (none) -> Murata; MPN (none) -> GRT188R61C106KE13D
- D2: DPN (none) -> 732-4971-1-ND; DST (none) -> Digi-Key; MFR (none) -> Wurth; MPN (none) -> 150060GS75000
- J1: DPN (none) -> 952-3875-1-ND; DST (none) -> Digi-Key; MFR (none) -> Harwin; MPN (none) -> M55-7011242R
- J2: DPN (none) -> H11891CT-ND; DST (none) -> Digi-Key; MFR (none) -> Hirose; MPN (none) -> U.FL-R-SMT-1(10)
- R1, R10, R3, R4, R5, R6, R7, R8, R9: DPN (none) -> RMCF0603FT4K70CT-ND; DST (none) -> Digi-Key; MFR (none) -> Stackpole Electronics Inc; MPN (none) -> RMCF0603FT4K70
- R11, R12, R2: DPN (none) -> RMCF0603FT2K70CT-ND; DST (none) -> Digi-Key; MFR (none) -> Stackpole Electronics Inc; MPN (none) -> RMCF0603FT2K70
- TP1, TP2, TP3, TP4, TP5, TP6, TP7, TP8: DPN (none) -> N/A; DST (none) -> N/A; MFR (none) -> N/A; MPN (none) -> N/A
- U1: DPN (none) -> LTC4305IGN#PBF-ND; DST (none) -> Digi-Key; MFR (none) -> Analog Devices; MPN (none) -> LTC4305IGN#PBF
- U2, U3: DPN (none) -> 1267-1072-1-ND; DST (none) -> Digi-Key; MFR (none) -> Memsic; MPN (none) -> MMC5883MA

Commit message: Added 3D models and fixed fab des
3D models of antenna patch (-Z) and M55 connector & magIc2 chip on both boards.
Changed lines of the file:
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@@
 (kicad_sch
-	(version 20231120)
+	(version 20250114)
 	(generator "eeschema")
-	(generator_version "8.0")
+	(generator_version "9.0")
 	(paper "B")
 	(title_block
@@
 		(rev "1.3")
 	)
+	(text "-X+Y Corner"
+		(exclude_from_sim no)
+		(at 332.74 184.15 0)
+		(effects
+			(font
+				(size 1.778 1.5113)
+			)
+			(justify left bottom)
+		)
+	)
+	(text "MAG-PWR"
+		(exclude_from_sim no)
+		(at 106.68 134.62 0)
+		(effects
+			(font
+				(size 1.27 1.27)
+			)
+			(justify left bottom)
+		)
+	)
+	(text "All resistors 0603 1% unless otherwise noted.\nAll capacitors 0603 x5R 16V or better unless otherwise noted."
+		(exclude_from_sim no)
+		(at 237.49 261.62 0)
+		(effects
+			(font
+				(size 1.27 1.27)
+			)
+			(justify left bottom)
+		)
+	)
+	(text "Stuff only if flying DxWiFi without deployable helical system."
+		(exclude_from_sim no)
+		(at 130.81 63.5 0)
+		(effects
+			(font
+				(size 1.27 1.27)
+			)
+		)
+	)
+	(text "Populate for flight? Or?"
+		(exclude_from_sim no)
+		(at 142.24 196.85 0)
+		(effects
+			(font
+				(size 1.27 1.27)
+			)
+		)
+	)
+	(text "Firmware: \"PZ2\""
+		(exclude_from_sim no)
+		(at 341.63 185.42 0)
+		(effects
+			(font
+				(size 1.27 1.27)
+			)
+		)
+	)
+	(text "+X-Y Corner"
+		(exclude_from_sim no)
+		(at 330.2 121.92 0)
+		(effects
+			(font
+				(size 1.778 1.5113)
+			)
+			(justify left bottom)
+		)
+	)
+	(text "ADRS2:ADRS0 = 000\ngives address 0x88"
+		(exclude_from_sim no)
+		(at 176.53 165.1 0)
+		(effects
+			(font
+				(size 1.27 1.27)
+			)
+		)
+	)
+	(text "Firmware: \"PZ1\""
+		(exclude_from_sim no)
+		(at 337.82 123.19 0)
+		(effects
+			(font
+				(size 1.27 1.27)
+			)
+		)
+	)
+	(text "3.3V and I2C signals are provide by the \nADCS card via the SPARE lines on the \nbackplane:\n\n   MAG-SDA = SPARE1 + SPARE2\n   MAG-SCL = SPARE3 + SPARE4 \n   MAG-PWR = SPARE5 + SPARE6.\n\nThese lines are delivered via the \n12 pin connector on the -Z end card"
+		(exclude_from_sim no)
+		(at 53.34 148.59 0)
+		(effects
+			(font
+				(size 1.27 1.27)
+			)
+			(justify left bottom)
+		)
+	)
+	(text "2.4 GHz backup antenna"
+		(exclude_from_sim no)
+		(at 128.27 67.31 0)
+		(effects
+			(font
+				(size 1.27 1.27)
+			)
+			(justify left bottom)
+		)
+	)
 	(junction
 		(at 233.68 171.45)
@@
 		)
 	)
-	(text "-X+Y Corner"
-		(exclude_from_sim no)
-		(at 332.74 184.15 0)
-		(effects
-			(font
-				(size 1.778 1.5113)
-			)
-			(justify left bottom)
-		)
-	)
-	(text "MAG-PWR"
-		(exclude_from_sim no)
-		(at 106.68 134.62 0)
-		(effects
-			(font
-				(size 1.27 1.27)
-			)
-			(justify left bottom)
-		)
-	)
-	(text "All resistors 0603 1% unless otherwise noted.\nAll capacitors 0603 x5R 16V or better unless otherwise noted."
-		(exclude_from_sim no)
-		(at 237.49 261.62 0)
-		(effects
-			(font
-				(size 1.27 1.27)
-			)
-			(justify left bottom)
-		)
-	)
-	(text "Stuff only if flying DxWiFi without deployable helical system."
-		(exclude_from_sim no)
-		(at 130.81 63.5 0)
-		(effects
-			(font
-				(size 1.27 1.27)
-			)
-		)
-	)
-	(text "Populate for flight? Or?"
-		(exclude_from_sim no)
-		(at 142.24 196.85 0)
-		(effects
-			(font
-				(size 1.27 1.27)
-			)
-		)
-	)
-	(text "Firmware: \"PZ2\""
-		(exclude_from_sim no)
-		(at 341.63 185.42 0)
-		(effects
-			(font
-				(size 1.27 1.27)
-			)
-		)
-	)
-	(text "+X-Y Corner"
-		(exclude_from_sim no)
-		(at 330.2 121.92 0)
-		(effects
-			(font
-				(size 1.778 1.5113)
-			)
-			(justify left bottom)
-		)
-	)
-	(text "ADRS2:ADRS0 = 000\ngives address 0x88"
-		(exclude_from_sim no)
-		(at 176.53 165.1 0)
-		(effects
-			(font
-				(size 1.27 1.27)
-			)
-		)
-	)
-	(text "Firmware: \"PZ1\""
-		(exclude_from_sim no)
-		(at 337.82 123.19 0)
-		(effects
-			(font
-				(size 1.27 1.27)
-			)
-		)
-	)
-	(text "3.3V and I2C signals are provide by the \nADCS card via the SPARE lines on the \nbackplane:\n\n   MAG-SDA = SPARE1 + SPARE2\n   MAG-SCL = SPARE3 + SPARE4 \n   MAG-PWR = SPARE5 + SPARE6.\n\nThese lines are delivered via the \n12 pin connector on the -Z end card"
-		(exclude_from_sim no)
-		(at 53.34 148.59 0)
-		(effects
-			(font
-				(size 1.27 1.27)
-			)
-			(justify left bottom)
-		)
-	)
-	(text "2.4 GHz backup antenna"
-		(exclude_from_sim no)
-		(at 128.27 67.31 0)
-		(effects
-			(font
-				(size 1.27 1.27)
-			)
-			(justify left bottom)
-		)
-	)
 	(label "SDA1"
 		(at 276.86 127 0)
-		(fields_autoplaced yes)
 		(effects
 			(font
@@
 	(label "MAG-SCL"
 		(at 106.68 129.54 0)
-		(fields_autoplaced yes)
 		(effects
 			(font
@@
 	(label "SCL2"
 		(at 214.63 134.62 0)
-		(fields_autoplaced yes)
 		(effects
 			(font
@@
 	(label "SCL1"
 		(at 276.86 124.46 0)
-		(fields_autoplaced yes)
 		(effects
 			(font
@@
 	(label "SCL2"
 		(at 276.86 186.69 0)
-		(fields_autoplaced yes)
 		(effects
 			(font
@@
 	(label "SDA2"
 		(at 214.63 137.16 0)
-		(fields_autoplaced yes)
 		(effects
 			(font
@@
 	(label "SCL1"
 		(at 214.63 124.46 0)
-		(fields_autoplaced yes)
 		(effects
 			(font
@@
 	(label "MAG-SDA"
 		(at 106.68 124.46 0)
-		(fields_autoplaced yes)
 		(effects
 			(font
@@
 	(label "MAG-SDA"
 		(at 160.02 132.08 0)
-		(fields_autoplaced yes)
 		(effects
 			(font
@@
 	(label "SDA1"
 		(at 214.63 127 0)
-		(fields_autoplaced yes)
 		(effects
 			(font
@@
 	(label "MAG-SCL"
 		(at 160.02 129.54 0)
-		(fields_autoplaced yes)
 		(effects
 			(font
@@
 	(label "SDA2"
 		(at 276.86 189.23 0)
-		(fields_autoplaced yes)
 		(effects
 			(font
@@
 	(label "GND"
 		(at 106.68 139.7 0)
-		(fields_autoplaced yes)
 		(effects
 			(font
@@
 		)
 	)
+	(embedded_fonts no)
 )
