File: oresat0.5-minusz-end-cap/oresat0.5-minusz-end-cap.kicad_pcb (KiCad board)
At the start: 2 copper layers, 105.6 x 105.6 mm, 48 parts, among them J1 M55-7011242R, J2 U.FL-R-SMA, U1 LTC4305, U2 MMC5983MA, U3 MMC5983MA

Commit message: Updated BOM to include MFR/MPN/etc.
Parts:
- removed the REF** at (167.5, 75.0)
- TP1, TP2, TP3, TP4, TP5, TP6, TP7, TP8: value TEST-POINT-LARGE-SQUARE -> Test-Point
