File: esi-minusz-end-cap/esi-minusZ-end-cap.kicad_sch (KiCad schematic)
At the start: 38 parts, among them J1 M55-7011242R, J2 U.FL-R-SMA, U1 RM3100, U2 RM3100

Commit message: New DFX & reposition GPS 7 magnetometers
Connections:
- net GND: now also J1.MP (SHIELD); no longer J1.SH (SHIELD)
Changed lines of the file:
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@@
 		(pin "9"
 		)
-		(pin "SH"
+		(pin "MP"
 		)
 		(instances

Commit message: ESI -Z end cap, with build files, final answer
Parts:
- J1: symbol oresat-connectors:J-HARWIN-M55-6001242R -> Connector_Generic_MountingPin:Conn_01x12_MountingPin
- L3, L4, L5, L7, L8, L9: DIS PNI -> N/A; DPN (none) -> N/A; MFR (none) -> PNI
- U1, U2: DIS PNI -> N/A; DPN RM3100 -> N/A; MFR (none) -> PNI; MPN (none) -> RM3100
Other:
- note added: "0805"
- note added: "All resistors 0603 1% and AEQ certified unless otherwise noted. All capacitors 0603 x5R 16V and AEQ certified or better unless otherwise noted."
- note removed: "All resistors 0603 1% unless otherwise noted. All capacitors 0603 x5R 16V or better unless otherwise noted."
