File: oresat1-minusz-end-cap/oresat1-minusZ-end-cap.kicad_sch (KiCad schematic)
At the start: 38 parts, among them J1 M55-7011242R, J2 U.FL-R-SMA, U1 RM3100, U2 RM3100

Commit message: Small changes
Requires layout work still
Changed lines of the file:
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@@
 		(dnp no)
 		(property "Reference" "R7"
-			(at 262.382 194.31 0)
+			(at 262.382 193.294 0)
 			(show_name no)
 			(do_not_autoplace no)
@@
 		)
 		(property "Value" "121"
-			(at 266.192 194.31 0)
+			(at 266.192 193.294 0)
 			(show_name no)
 			(do_not_autoplace no)

Commit message: Pushed for design review
Connections:
- net at R7.1, U2.8 (ZINN): now also L5.1; no longer L5.2
- net at R6.1, U2.7 (ZINP): now also L5.2; no longer L5.1
- net at R14.1, U1.7 (ZINP): now also L9.2; no longer L9.1
- net at R15.1, U1.8 (ZINN): now also L9.1; no longer L9.2
Other:
- note added: "Z-axis inverted to compensate for position in satellite"
- moved on the sheet: L5, L9
Changed lines of the file:
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@@
 		)
 	)
+	(text "Z-axis inverted to compensate for position in satellite"
+		(exclude_from_sim no)
+		(at 302.26 197.104 0)
+		(effects
+			(font
+				(size 1.27 1.27)
+			)
+		)
+	)
 	(text "MAG-PWR"
 		(exclude_from_sim no)
@@
 		)
 	)
+	(text "Z-axis inverted to compensate for position in satellite"
+		(exclude_from_sim no)
+		(at 302.514 99.314 0)
+		(effects
+			(font
+				(size 1.27 1.27)
+			)
+		)
+	)
 	(text "DRVP/DRVN TRACES MUST BE EXACT EQUAL LENGTH PER SENSOR COUPLE"
 		(exclude_from_sim no)
@@
 	(symbol
 		(lib_id "Device:L")
-		(at 274.32 193.04 0)
+		(at 274.32 193.04 180)
 		(unit 1)
 		(body_style 1)
@@
 					(size 1.27 1.27)
 				)
-				(justify left)
+				(justify right)
 			)
 		)
@@
 					(size 1.27 1.27)
 				)
-				(justify left)
+				(justify right)
 			)
 		)
@@
 	(symbol
 		(lib_id "Device:L")
-		(at 274.32 95.25 0)
+		(at 274.32 95.25 180)
 		(unit 1)
 		(body_style 1)
@@
 					(size 1.27 1.27)
 				)
-				(justify left)
+				(justify right)
 			)
 		)
@@
 					(size 1.27 1.27)
 				)
-				(justify left)
+				(justify right)
 			)
 		)

Commit message: routine push
Changed lines of the file:
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@@
 	)
 	(junction
-		(at 245.11 40.64)
-		(diameter 0)
-		(color 0 0 0 0)
-	)
-	(junction
 		(at 229.87 172.72)
 		(diameter 0)
@@
 	)
 	(junction
+		(at 245.11 40.64)
+		(diameter 0)
+		(color 0 0 0 0)
+	)
+	(junction
 		(at 240.03 40.64)
 		(diameter 0)
@@
 	)
 	(junction
-		(at 245.11 138.43)
-		(diameter 0)
-		(color 0 0 0 0)
-	)
-	(junction
 		(at 163.83 118.11)
 		(diameter 0)
@@
 	)
 	(junction
+		(at 245.11 138.43)
+		(diameter 0)
+		(color 0 0 0 0)
+	)
+	(junction
 		(at 214.63 138.43)
 		(diameter 0)
@@
 	(wire
 		(pts
-			(xy 247.65 138.43) (xy 245.11 138.43)
+			(xy 250.19 138.43) (xy 245.11 138.43)
 		)
 		(stroke
@@
 	(wire
 		(pts
-			(xy 247.65 54.61) (xy 247.65 40.64)
+			(xy 250.19 54.61) (xy 250.19 40.64)
 		)
 		(stroke
@@
 	(wire
 		(pts
-			(xy 247.65 152.4) (xy 247.65 138.43)
+			(xy 250.19 152.4) (xy 250.19 138.43)
 		)
 		(stroke
@@
 	(wire
 		(pts
-			(xy 245.11 40.64) (xy 247.65 40.64)
+			(xy 245.11 40.64) (xy 250.19 40.64)
 		)
 		(stroke
@@
 		(in_pos_files yes)
 		(dnp no)
-		(fields_autoplaced yes)
 		(property "Reference" "U2"
-			(at 249.7933 149.86 0)
+			(at 250.952 150.114 0)
 			(show_name no)
 			(do_not_autoplace no)
@@
 		)
 		(property "Value" "RM3100"
-			(at 249.7933 152.4 0)
+			(at 250.952 151.892 0)
 			(show_name no)
 			(do_not_autoplace no)
@@
 		(in_pos_files yes)
 		(dnp no)
-		(fields_autoplaced yes)
 		(property "Reference" "U1"
-			(at 249.7933 52.07 0)
+			(at 251.714 51.816 0)
 			(show_name no)
 			(do_not_autoplace no)
@@
 		)
 		(property "Value" "RM3100"
-			(at 249.7933 54.61 0)
+			(at 251.714 54.356 0)
 			(show_name no)
 			(do_not_autoplace no)
