File: oresat1-minusz-end-cap/oresat1-minusZ-end-cap.kicad_sch (KiCad schematic)
At the start: 38 parts, among them J1 M55-7011242R, J2 U.FL-R-SMA, U1 RM3100, U2 RM3100

Commit message: routine push
Parts:
- added R16, R17, R18, R19: 121, oresat-passives:0603-C-NOSILK, symbol oresat-passives:R-US
Connections:
- net +3.3v: now also R16.1, R18.1; no longer U1.28 (MISO/SA1)
- net GND: now also R17.2, R19.2; no longer U1.3 (SSN/SA0)
- new net: R18.2, R19.1, U1.3 (SSN/SA0)
- new net: R16.2, R17.1, U1.28 (MISO/SA1)

Commit message: Brought -Z end cap up to the current state. Added address resistors, fixed capacitor placement, polished and made PNI layout consistent, added makefile and readme.
Parts:
- added FID101, FID102, FID103, FID104, FID105, FID106: Fiducial, Fiducial:Fiducial_1mm_Mask2mm, symbol Mechanical:Fiducial
- added R20, R21, R22, R23: 121, oresat-passives:0603-C-NOSILK, symbol oresat-passives:R-US
- J1: footprint oresat-connectors:J-Harwin-M55-60X1242R -> oresat-connectors:J-Harwin-M55-7XX1242R; symbol oresat-connectors:J-HARWIN-M55-6001242R -> Connector_Generic_MountingPin:Conn_01x12_MountingPin
- R18: now fitted
- R19: now not fitted
- U1, U2: footprint oresat-misc:RM3100-MagI2C -> oresat-ics:U-PNI-RM3100-IC
Connections:
- net +3.3v: now also R20.1, R22.1
- net GND: now also J1.MP (MountPin), R21.2, R23.2; no longer J1.SH (SHIELD), U2.28 (MISO/SA1), U2.3 (SSN/SA0)
- net MAG-SCL: now also U1.27 (SCLK), U2.27 (SCLK); no longer U1.1 (MOSI/SDA), U2.1 (MOSI/SDA)
- net MAG-SDA: now also U1.1 (MOSI/SDA), U2.1 (MOSI/SDA); no longer U1.27 (SCLK), U2.27 (SCLK)
- new net: R22.2, R23.1, U2.3 (SSN/SA0)
- new net: R20.2, R21.1, U2.28 (MISO/SA1)
Other:
- note added: "-Z+X-Y Corner"
- note added: "-Z-X+Y Corner"
- note added: "0805"
- note added: "Address: 10"
- note added: "Address: 11"
- note added: "All resistors 0603 1% and AEQ unless otherwise noted. All capacitors 0603 10% X5R Wv >= 25V and AEQ or better unless otherwise noted."
- note added: "Back Fiducials"
- note added: "DRVP/DRVN TRACES SHOULD BE EQUAL LENGTH PER SENSOR COUPLE"
- note added: "Front Fiducials"
- note added: "Z sensor is inverted since we're on the top of the PCB, and the sensor is tuned for North/East/Down."
- note removed: "+X-Y Corner"
- note removed: "-X+Y Corner"
- note removed: "Address: 00"
- note removed: "Address: 01"
- note removed: "All resistors 0603 1% unless otherwise noted. All capacitors 0603 x5R 16V or better unless otherwise noted."
- note removed: "DRVP/DRVN TRACES MUST BE EXACT EQUAL LENGTH PER SENSOR COUPLE"
- note removed: "Z-axis inverted to compensate for position in satellite"
- moved on the sheet: C6, TP3, TP6, TP7, TP8

Commit message: Bring BOM up to date
Parts:
- L3: value SEN2-XY (y-axis) -> RM3100-XY; DIS PNI -> N/A; DPN (none) -> N/A; MFR (none) -> PNI Sensors; MPN (none) -> PN13104
- L4: value SEN2-XY (x-axis) -> RM3100-XY; DIS PNI -> N/A; DPN (none) -> N/A; MFR (none) -> PNI Sensors; MPN (none) -> PN13104
- L5: value SEN2-Z (z-axis) -> RM3100-Z; DIS PNI -> N/A; DPN (none) -> N/A; MFR (none) -> PNI Sensors; MPN (none) -> PN13101
- L7: value SEN1-XY (x-axis) -> RM3100-XY; DIS PNI -> N/A; DPN (none) -> N/A; MFR (none) -> PNI Sensors; MPN (none) -> PN13104
- L8: value SEN1-XY (y-axis) -> RM3100-XY; DIS PNI -> N/A; DPN (none) -> N/A; MFR (none) -> PNI Sensors; MPN (none) -> PN13104
- L9: value SEN1-Z (z-axis) -> RM3100-Z; DIS PNI -> N/A; DPN (none) -> N/A; MFR (none) -> PNI Sensors; MPN (none) -> PN13101
- U1, U2: DIS PNI -> N/A; DPN RM3100 -> N/A; MFR (none) -> PNI Sensors; MPN (none) -> PN13156

Commit message: Spelling mistakes and better I2C documentation
Other:
- note added: "Address bits: 10"
- note added: "Address bits: 11"
- note added: "I2C Address: 0x22"
- note added: "I2C Address: 0x23"
- note removed: "Address: 10"
- note removed: "Address: 11"
Changed lines of the file:
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@@
 		)
 	)
-	(text "Address: 10"
+	(text "I2C Address: 0x22"
 		(exclude_from_sim no)
 		(at 276.352 150.876 0)
@@
 		)
 	)
-	(text "Address: 10"
+	(text "Address bits: 10"
 		(exclude_from_sim no)
-		(at 226.06 180.594 0)
+		(at 222.504 180.594 0)
 		(effects
 			(font
@@
 		)
 	)
-	(text "Address: 11"
+	(text "Address bits: 11"
 		(exclude_from_sim no)
-		(at 217.17 82.55 0)
+		(at 221.742 82.55 0)
 		(effects
 			(font
@@
 		)
 	)
-	(text "Address: 11"
+	(text "I2C Address: 0x23"
 		(exclude_from_sim no)
 		(at 275.082 57.15 0)
