File: oresat1-plusz-end-cap/oresat1-plusz-end-cap.kicad_pcb (KiCad board)
At the start: 4 copper layers, 105.6 x 105.6 mm, 63 parts, among them J1 M55-7011242R, J2 U.FL-R-SMA, U1 RM3100, U2 RM3100

Commit message: v1.1 +Z end cap with polishing fixes
Parts:
- moved J2 0.47 mm to (191.9, 78.2)
Other:
- board text added: "WE'RE GOING TO 0x20!!!!"
